File: Velox.kicad_sch (KiCad schematic)
At the start: 4 parts, among them J1 Conn_Coaxial, J2 OLED, U1 MOUDLE-SEEEDUINO-XIAO-ESP32C3, U2 Ai-Thinker-Ra-01

Commit message: Polished design
Parts:
- added Cap1, Cap2: C, Capacitor_SMD:C_0805_2012Metric_Pad1.18x1.45mm_HandSolder, symbol Device:C
- added IND1: L, Inductor_SMD:L_0805_2012Metric_Pad1.15x1.40mm_HandSolder, symbol Device:L
- renumbered U1 to ESP32C3, U2 to LoRa-RA-01, J2 to OLED1, J1 to SMA1
Connections:
- net ANT: now also Cap1.1, IND1.1; no longer SMA1.1 (In)
- net D3: now also LoRa-RA-01.6 (DIO1)
- net GND: now also Cap1.2, Cap2.2
- new net: Cap2.1, IND1.2, SMA1.1 (In)
- no-connect marks 5 -> 4
